File: Negligence.kicad_pcb (KiCad board)
At the start: 2 copper layers, 228.9 x 105.7 mm, 121 parts, among them J1 AVR-ISP-6, SW1 keyboard_parts_KEYSW, SW10 keyboard_parts_KEYSW, SW11 keyboard_parts_KEYSW, SW12 keyboard_parts_KEYSW, SW13 keyboard_parts_KEYSW, SW14 keyboard_parts_KEYSW, SW15 keyboard_parts_KEYSW, SW16 keyboard_parts_KEYSW, SW17 keyboard_parts_KEYSW, SW18 keyboard_parts_KEYSW, SW19 keyboard_parts_KEYSW, SW2 keyboard_parts_KEYSW, SW20 keyboard_parts_KEYSW, SW21 keyboard_parts_KEYSW, SW22 keyboard_parts_KEYSW, SW23 keyboard_parts_KEYSW, SW24 keyboard_parts_KEYSW, SW25 keyboard_parts_KEYSW, SW26 keyboard_parts_KEYSW, SW27 keyboard_parts_KEYSW, SW28 keyboard_parts_KEYSW, SW29 keyboard_parts_KEYSW, SW3 keyboard_parts_KEYSW, SW30 keyboard_parts_KEYSW, SW31 keyboard_parts_KEYSW, SW32 keyboard_parts_KEYSW, SW33 keyboard_parts_KEYSW, SW34 keyboard_parts_KEYSW, SW35 keyboard_parts_KEYSW, SW36 keyboard_parts_KEYSW, SW37 keyboard_parts_KEYSW, SW38 keyboard_parts_KEYSW, SW39 keyboard_parts_KEYSW, SW4 keyboard_parts_KEYSW, SW40 keyboard_parts_KEYSW, SW41 keyboard_parts_KEYSW, SW42 keyboard_parts_KEYSW, SW43 keyboard_parts_KEYSW, SW44 keyboard_parts_KEYSW, SW45 keyboard_parts_KEYSW, SW46 keyboard_parts_KEYSW, SW47 RESET, SW48 BOOT, SW5 keyboard_parts_KEYSW, SW6 keyboard_parts_KEYSW, SW7 keyboard_parts_KEYSW, SW8 keyboard_parts_KEYSW, SW9 keyboard_parts_KEYSW, Y1 16MHz

Commit message: CSV/gerber
Parts:
- added R7: 220Ω, cftkb:R_Axial_DIN0204_L3.6mm_D1.6mm_P7.62mm_Horizontal, F.Cu at (158.6, 69.3)
- added R8: 220Ω, cftkb:R_Axial_DIN0204_L3.6mm_D1.6mm_P7.62mm_Horizontal, F.Cu at (158.6, 66.5)
- added R9: 220Ω, cftkb:R_Axial_DIN0204_L3.6mm_D1.6mm_P7.62mm_Horizontal, F.Cu at (158.6, 63.6)
- added RGB LED: LED_RGBA, LED_THT:LED_D5.0mm-4_RGB, F.Cu at (123.4, 54.5)
- renumbered USB to USB1
Routing:
- net Net-(D49-Pad1): track 0.00 -> 46.4 mm
- net Net-(D49-Pad2): track 0.00 -> 42.7 mm
- net Net-(D49-Pad3): track 0.00 -> 38.5 mm
- net +5V: track 92.9 -> 130.1 mm
- net GND: track 100.8 -> 106.5 mm, vias 23 -> 24
- net /ROW3: track 175.2 -> 176.0 mm
- net /RESET: track 107.4 -> 107.2 mm, vias 0 -> 1

Commit message: Add addressable led
Parts:
- removed R7, R8, R9: 220Ω, cftkb:R_Axial_DIN0204_L3.6mm_D1.6mm_P7.62mm_Horizontal
- removed REF** (x9): MountingHole_2.2mm_M2_Pad, cftkb:MountingHole_2.2mm_M2_Pad
- removed RGB LED: LED_RGBA, LED_THT:LED_D5.0mm-4_RGB
- added H1: MountingHole, MountingHole:MountingHole_2.2mm_M2, F.Cu at (17.0, 74.9)
- added H2: MountingHole, MountingHole:MountingHole_2.2mm_M2, F.Cu at (238.3, 54.0)
- added H3: MountingHole, MountingHole:MountingHole_2.2mm_M2, F.Cu at (128.5, 117.5)
- added H4: MountingHole, MountingHole:MountingHole_2.2mm_M2, F.Cu at (51.4, 98.4)
- added H5: MountingHole, MountingHole:MountingHole_2.2mm_M2, F.Cu at (17.0, 54.1)
- added H6: MountingHole, MountingHole:MountingHole_2.2mm_M2, F.Cu at (223.9, 98.4)
- added H7: MountingHole, MountingHole:MountingHole_2.2mm_M2, F.Cu at (224.2, 136.5)
- added H8: MountingHole, MountingHole:MountingHole_2.2mm_M2, F.Cu at (238.5, 74.9)
- added H9: MountingHole, MountingHole:MountingHole_2.2mm_M2, F.Cu at (51.3, 136.5)
- added LED: SK6812, LED_SMD:LED_SK6812_PLCC4_5.0x5.0mm_P3.2mm, F.Cu at (197.4, 71.9)
- renumbered ATmega328P-PU to U1
Connections:
- U1 pad 12: Net-(U1-Pad12) -> /RGB_LED
Routing:
- net Net-(D49-Pad1): track 46.4 -> 0.00 mm
- net Net-(D49-Pad2): track 42.7 -> 0.00 mm
- net Net-(D49-Pad3): track 38.5 -> 0.00 mm
- net +5V: track 130.1 -> 98.1 mm
- net /RGB_LED: track 0.00 -> 16.2 mm
- net GND: track 106.5 -> 100.8 mm
